File: board/board.kicad_pcb (KiCad board)
At the start: 2 copper layers, 21 x 13 mm, 1 part

Commit message: initial
Parts:
- added C1: 10uF, Capacitor_SMD:C_0603_1608Metric, F.Cu at (154.2, 93.3)
- added C2: 10uF, Capacitor_SMD:C_0603_1608Metric, F.Cu at (154.2, 94.8)
- added J1: 003_power, on_edge:on_edge_2x05_device, F.Cu at (140.0, 96.5)
- added J2: Conn_01x02_Male, Connector_PinHeader_2.54mm:PinHeader_1x02_P2.54mm_Vertical, F.Cu at (146.8, 94.8)
- added J3: 003_power, on_edge:on_edge_2x05_host, F.Cu at (161.0, 96.5)
- added L1: 4.7uH, Inductor_SMD:L_0805_2012Metric, F.Cu at (150.5, 93.3)
- added R1: 10k, Resistor_SMD:R_0603_1608Metric, F.Cu at (146.8, 97.0)
- added R2: 1M, Resistor_SMD:R_0603_1608Metric, F.Cu at (154.2, 96.3)
- added R3: 180k, Resistor_SMD:R_0603_1608Metric, F.Cu at (154.2, 97.8)
- added U1: TLV61220, Package_TO_SOT_SMD:SOT-23-6, F.Cu at (150.5, 96.0)
- LOGO1: moved to B.Cu
- turned LOGO1 to 180 degrees
Routing:
- net GND: track 0.00 -> 29.9 mm
- net /implementation/in: track 0.00 -> 17.0 mm, vias 0 -> 2
- net /implementation/3.3V: track 0.00 -> 11.2 mm, vias 0 -> 1
- net /implementation/EN: track 0.00 -> 4.29 mm
- net Net-(R2-Pad2): track 0.00 -> 3.15 mm
- net Net-(L1-Pad2): track 0.00 -> 1.77 mm
Other:
- outline, holes or cut-outs redrawn
- board text added: "enable"
- board text added: "osf.003"
- board text added: "osf.b100.v0.1"
